File: wave_light_lp5569.sch (KiCad schematic (older format))
At the start: 25 parts, among them J1 Conn_01x06_Male, J10 Conn_01x02_Male, J11 Conn_01x02_Male, J12 Conn_01x02_Male, J13 Conn_01x02_Male, J14 Conn_01x02_Male, J2 Conn_02x04_Odd_Even, J3 Conn_01x06_Female, J4 Conn_01x03_Male, J5 Conn_01x02_Male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

Commit message: First go at a wedge-shaped board
Parts:
- removed J10, J11, J12, J13, J5, J6, J7, J8, J9: Conn_01x02_Male, Connector_JST:JST_XH_B2B-XH-A_1x02_P2.50mm_Vertical, symbol Connector:Conn_01x02_Male
- removed J2: Conn_02x04_Odd_Even, Pin_Headers:Pin_Header_Straight_2x04_Pitch2.54mm, symbol Connector_Generic:Conn_02x04_Odd_Even
- removed J4: Conn_01x03_Male, Pin_Headers:Pin_Header_Straight_1x03_Pitch2.54mm, symbol Connector:Conn_01x03_Male
- added H1, H2, H3: MountingHole, MountingHole:MountingHole_2.7mm, symbol Mechanical:MountingHole
- added J2, J5: Conn_01x09_Male, Connector_JST:JST_PH_B9B-PH-K_1x09_P2.00mm_Vertical, symbol Connector:Conn_01x09_Male
- added JP1, JP2, JP3, JP4: SolderJumper_2_Open, Jumper:SolderJumper-2_P1.3mm_Open_RoundedPad1.0x1.5mm, symbol Jumper:SolderJumper_2_Open
- added JP5: SolderJumper_3_Bridged12, Jumper:SolderJumper-3_P1.3mm_Bridged12_RoundedPad1.0x1.5mm, symbol Jumper:SolderJumper_3_Bridged12
- J1: footprint Pin_Headers:Pin_Header_Angled_1x06_Pitch2.54mm -> Connector_JST:JST_PH_B6B-PH-K_1x06_P2.00mm_Vertical
- J3: value Conn_01x06_Female -> Conn_01x06_Male; footprint Pin_Headers:Pin_Header_Angled_1x06_Pitch2.54mm -> Connector_JST:JST_PH_B6B-PH-K_1x06_P2.00mm_Vertical; symbol Connector:Conn_01x06_Female -> Connector:Conn_01x06_Male
Connections:
- net ADDR: now also JP1.2 (B), JP2.2 (B), JP3.2 (B), JP4.2 (B)
- net CLK: now also J3.4 (Pin_4); no longer J3.3 (Pin_3)
- net EN_PWM: now also J3.3 (Pin_3); no longer J3.4 (Pin_4)
- net GND: now also J3.6 (Pin_6), JP1.1 (A); no longer J3.1 (Pin_1)
- net GPIO_TRIG_INT: now also J3.5 (Pin_5); no longer J3.2 (Pin_2)
- net LED0: now also J5.1 (Pin_1)
- net LED1: now also J5.2 (Pin_2)
- net LED2: now also J5.3 (Pin_3)
- net LED3: now also J5.4 (Pin_4)
- net LED4: now also J5.5 (Pin_5)
- net LED5: now also J5.6 (Pin_6)
- net LED6: now also J5.7 (Pin_7)
- net LED7: now also J5.8 (Pin_8)
- net LED8: now also J5.9 (Pin_9)
- net SCL: now also J3.1 (Pin_1), JP2.1 (A); no longer J3.6 (Pin_6)
- net SDA: now also J3.2 (Pin_2), JP3.1 (A); no longer J3.5 (Pin_5)
- net VIN: now also JP4.1 (A), JP5.1 (A)
- net VLED: now also J2.1 (Pin_1), J2.2 (Pin_2), J2.3 (Pin_3), J2.4 (Pin_4), J2.5 (Pin_5), J2.6 (Pin_6), J2.7 (Pin_7), J2.8 (Pin_8), J2.9 (Pin_9), JP5.2 (C)
- net VOUT: now also JP5.3 (B)
Other:
- note added: "TODO: \nFigure out external clock; internal clock doesn't want to come out the clock pin\n\n"

Commit message: Checkpointing work on the wedge board
Parts:
- H1, H2, H3: footprint MountingHole:MountingHole_2.7mm -> MountingHole:MountingHole_2.7mm_Pad
Changed lines of the file:
@@
 F 0 "H1" H 8340 2176 50  0000 L CNN
 F 1 "MountingHole" H 8340 2085 50  0000 L CNN
-F 2 "MountingHole:MountingHole_2.7mm" H 8240 2130 50  0001 C CNN
+F 2 "MountingHole:MountingHole_2.7mm_Pad" H 8240 2130 50  0001 C CNN
 F 3 "~" H 8240 2130 50  0001 C CNN
 	1    8240 2130
@@
 F 0 "H2" H 8340 2366 50  0000 L CNN
 F 1 "MountingHole" H 8340 2275 50  0000 L CNN
-F 2 "MountingHole:MountingHole_2.7mm" H 8240 2320 50  0001 C CNN
+F 2 "MountingHole:MountingHole_2.7mm_Pad" H 8240 2320 50  0001 C CNN
 F 3 "~" H 8240 2320 50  0001 C CNN
 	1    8240 2320
@@
 F 0 "H3" H 8340 2556 50  0000 L CNN
 F 1 "MountingHole" H 8340 2465 50  0000 L CNN
-F 2 "MountingHole:MountingHole_2.7mm" H 8240 2510 50  0001 C CNN
+F 2 "MountingHole:MountingHole_2.7mm_Pad" H 8240 2510 50  0001 C CNN
 F 3 "~" H 8240 2510 50  0001 C CNN
 	1    8240 2510

Commit message: Finally passing ERC and DRC, seems ready to send off for fab
Parts:
- removed C3: 1uF, Capacitors_SMD:C_0805_HandSoldering, symbol Device:C
- removed J2, J5: Conn_01x09_Male, Connector_JST:JST_PH_B9B-PH-K_1x09_P2.00mm_Vertical, symbol Connector:Conn_01x09_Male
- added J2: Conn_02x09_Odd_Even, Connector_PinHeader_2.54mm:PinHeader_2x09_P2.54mm_Horizontal, symbol Connector_Generic:Conn_02x09_Odd_Even
- H1, H2: value MountingHole -> MountingHole_Pad; symbol Mechanical:MountingHole -> Mechanical:MountingHole_Pad
- H3: value MountingHole -> MountingHole_pad; symbol Mechanical:MountingHole -> Mechanical:MountingHole_Pad
- J1, J3: value Conn_01x06_Male -> Conn_01x07_Male; footprint Connector_JST:JST_PH_B6B-PH-K_1x06_P2.00mm_Vertical -> Connector_JST:JST_PH_B7B-PH-K_1x07_P2.00mm_Vertical; symbol Connector:Conn_01x06_Male -> Connector:Conn_01x07_Male
- J4: renamed from J14; footprint Connector_JST:JST_XH_B2B-XH-A_1x02_P2.50mm_Vertical -> Connector_JST:JST_XH_S2B-XH-A_1x02_P2.50mm_Horizontal
Connections:
- net GND: now also H1.1, H2.1, H3.1, J1.7 (Pin_7), J3.7 (Pin_7); no longer J1.6 (Pin_6), J3.6 (Pin_6)
- net LED0: now also J2.1 (Pin_1)
- net LED1: now also J2.3 (Pin_3)
- net LED2: now also J2.5 (Pin_5)
- net LED3: now also J2.7 (Pin_7)
- net LED4: now also J2.9 (Pin_9)
- net LED5: now also J2.11 (Pin_11)
- net LED6: now also J2.13 (Pin_13)
- net LED7: now also J2.15 (Pin_15)
- net LED8: now also J2.17 (Pin_17)
- net VIN: now also J1.6 (Pin_6), J3.6 (Pin_6)
- net VLED: now also J2.10 (Pin_10), J2.12 (Pin_12), J2.14 (Pin_14), J2.16 (Pin_16), J2.18 (Pin_18), J2.2 (Pin_2), J2.4 (Pin_4), J2.6 (Pin_6), J2.8 (Pin_8)
Other:
- note added: "Power Input"
- note removed: "TODO: \nFigure out external clock; internal clock doesn't want to come out the clock pin\n\n"

Commit message: Final version, sent to fab
Parts:
- added R4: 120k, Resistor_SMD:R_0805_2012Metric, symbol Device:R_US
- C1, C2, C4, C5, C6: footprint Capacitors_SMD:C_0805_HandSoldering -> Capacitor_SMD:C_0805_2012Metric
- R1, R2, R3: footprint Resistors_SMD:R_0805_HandSoldering -> Resistor_SMD:R_0805_2012Metric
- U1: footprint TO_SOT_Packages_SMD:SOT-23-5_HandSoldering -> Package_TO_SOT_SMD:SOT-23-5
Connections:
- net CLK: now also R4.2
- net VIN: now also R4.1
Other:
- note added: "CLK Pullup"
- note added: "Only populate R1-R4 on first board"
- note removed: "Only populate on first board"
Changed lines of the file:
@@
 F 0 "C4" H 5900 1900 50  0000 R CNN
 F 1 "1uF" H 5900 2000 50  0000 R CNN
-F 2 "Capacitors_SMD:C_0805_HandSoldering" H 5888 2100 50  0001 C CNN
+F 2 "Capacitor_SMD:C_0805_2012Metric" H 5888 2100 50  0001 C CNN
 F 3 "~" H 5850 2250 50  0001 C CNN
 	1    5850 2250
@@
 F 0 "C5" H 6300 1900 50  0000 R CNN
 F 1 "1uF" H 6300 2000 50  0000 R CNN
-F 2 "Capacitors_SMD:C_0805_HandSoldering" H 6288 2100 50  0001 C CNN
+F 2 "Capacitor_SMD:C_0805_2012Metric" H 6288 2100 50  0001 C CNN
 F 3 "~" H 6250 2250 50  0001 C CNN
 	1    6250 2250
@@
 F 0 "U1" H 2750 2915 50  0000 C CNN
 F 1 "LP3990" H 2750 2824 50  0000 C CNN
-F 2 "TO_SOT_Packages_SMD:SOT-23-5_HandSoldering" H 2750 2850 50  0001 C CNN
+F 2 "Package_TO_SOT_SMD:SOT-23-5" H 2750 2850 50  0001 C CNN
 F 3 "" H 2750 2450 50  0001 C CNN
 	1    2750 2450
@@
 F 0 "C1" H 1885 2404 50  0000 R CNN
 F 1 "1uF" H 1885 2495 50  0000 R CNN
-F 2 "Capacitors_SMD:C_0805_HandSoldering" H 2038 2300 50  0001 C CNN
+F 2 "Capacitor_SMD:C_0805_2012Metric" H 2038 2300 50  0001 C CNN
 F 3 "~" H 2000 2450 50  0001 C CNN
 	1    2000 2450
@@
 F 0 "C2" H 3335 2404 50  0000 R CNN
 F 1 "1uF" H 3335 2495 50  0000 R CNN
-F 2 "Capacitors_SMD:C_0805_HandSoldering" H 3488 2300 50  0001 C CNN
+F 2 "Capacitor_SMD:C_0805_2012Metric" H 3488 2300 50  0001 C CNN
 F 3 "~" H 3450 2450 50  0001 C CNN
 	1    3450 2450
@@
 F 0 "R1" H 4918 1246 50  0000 L CNN
 F 1 "120k" H 4918 1155 50  0000 L CNN
-F 2 "Resistors_SMD:R_0805_HandSoldering" V 4890 1190 50  0001 C CNN
+F 2 "Resistor_SMD:R_0805_2012Metric" V 4890 1190 50  0001 C CNN
 F 3 "~" H 4850 1200 50  0001 C CNN
 	1    4850 1200
@@
 F 0 "C6" H 6885 3204 50  0000 R CNN
 F 1 "1uF" H 6885 3295 50  0000 R CNN
-F 2 "Capacitors_SMD:C_0805_HandSoldering" H 7038 3100 50  0001 C CNN
+F 2 "Capacitor_SMD:C_0805_2012Metric" H 7038 3100 50  0001 C CNN
 F 3 "~" H 7000 3250 50  0001 C CNN
 	1    7000 3250
@@
 F 0 "R2" H 5718 1246 50  0000 L CNN
 F 1 "2.2k" H 5718 1155 50  0000 L CNN
-F 2 "Resistors_SMD:R_0805_HandSoldering" V 5690 1190 50  0001 C CNN
+F 2 "Resistor_SMD:R_0805_2012Metric" V 5690 1190 50  0001 C CNN
 F 3 "~" H 5650 1200 50  0001 C CNN
 	1    5650 1200
@@
 F 0 "R3" H 6068 1246 50  0000 L CNN
 F 1 "2.2k" H 6068 1155 50  0000 L CNN
-F 2 "Resistors_SMD:R_0805_HandSoldering" V 6040 1190 50  0001 C CNN
+F 2 "Resistor_SMD:R_0805_2012Metric" V 6040 1190 50  0001 C CNN
 F 3 "~" H 6000 1200 50  0001 C CNN
 	1    6000 1200
@@
 GPIO Pullup
 Text Notes 4750 850  0    50   ~ 0
-Only populate on first board
+Only populate R1-R4 on first board
 Text Notes 1890 3820 0    50   ~ 0
 32h and 40h
@@
 	8140 2510 8140 2610
 Connection ~ 8140 2510
+$Comp
+L Device:R_US R4
+U 1 1 5FEA6400
+P 4850 1840
+F 0 "R4" H 4918 1886 50  0000 L CNN
+F 1 "120k" H 4918 1795 50  0000 L CNN
+F 2 "Resistor_SMD:R_0805_2012Metric" V 4890 1830 50  0001 C CNN
+F 3 "~" H 4850 1840 50  0001 C CNN
+	1    4850 1840
+	1    0    0    -1
+$EndComp
+Text GLabel 4750 1690 0    50   Input ~ 0
+VIN
+Wire Wire Line
+	4750 1690 4850 1690
+Text GLabel 4750 1990 0    50   Input ~ 0
+CLK
+Wire Wire Line
+	4750 1990 4850 1990
+Text Notes 4500 1590 0    50   ~ 0
+CLK Pullup
 $EndSCHEMATC
